File: NavKF.kicad_pcb (KiCad board)
At the start: 2 copper layers, 89 parts, among them J1 USB_C_Receptacle_USB2.0_16P, J2 USB_C_Receptacle_USB2.0_16P, Q1 BC817, SW1 Reset, SW2 Reset, U1 LAN8742A, U2 STMPS2141STR, U2 USBLC6-4SC6, U3 STM32H723ZGTx, U4 LAN8742A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

Commit message: KiCad: update NavKF
Parts:
- removed C1, C2, C4, C44, C7: 100nF, Capacitor_SMD:C_0402_1005Metric
- removed C3, C6: 10uF, Capacitor_SMD:C_0603_1608Metric
- removed C37, C38: 22pF, Capacitor_SMD:C_0603_1608Metric_Pad1.08x0.95mm_HandSolder
- removed C39: 100nF, Capacitor_SMD:C_0603_1608Metric_Pad1.08x0.95mm_HandSolder
- removed C45, C46: 22pF, Capacitor_SMD:C_0402_1005Metric
- removed C5: 470pF, Capacitor_SMD:C_0402_1005Metric
- removed C8: 4.7uF, Capacitor_SMD:C_0603_1608Metric
- removed D2: ESDALC6V1, Diode_SMD:D_SOD-882
- removed D6: ESD5Zxx, Diode_SMD:D_SOD-523
- removed FB2: 600R@100MHz, Inductor_SMD:L_0603_1608Metric
- removed J1, J2: USB_C_Receptacle_USB2.0_16P, MyLib_Connectors:GCT_USB4930-00-A_REVA
- removed R1, R10, R11, R2: 33R, Resistor_SMD:R_0402_1005Metric
- removed R12: 0R, Resistor_SMD:R_0402_1005Metric
- removed R13, R14, R37, R38: 49R9, Resistor_SMD:R_0402_1005Metric
- removed the R15 at (14.3, 76.6)
- removed the R16 at (14.3, 78.5)
- removed the R17 at (14.3, 80.5)
- removed the R18 at (55.3, 85.6)
- removed the R19 at (55.3, 87.5)
- removed R21, R22, R29: 10K, Resistor_SMD:R_0603_1608Metric
- removed R23: 33R, Resistor_SMD:R_0603_1608Metric
- removed R3, R4, R5, R6, R8: 10K, Resistor_SMD:R_0402_1005Metric
- removed R30, R31: 49.9Ω, Resistor_SMD:R_0603_1608Metric
- removed R7: 1K5, Resistor_SMD:R_0402_1005Metric
- removed R9: 12K1, Resistor_SMD:R_0402_1005Metric
- removed SW2: Reset, Button_Switch_SMD:SW_Tactile_SPST_NO_Straight_CK_PTS636Sx25SMTRLFS
- removed U1: LAN8742A, Package_DFN_QFN:VQFN-24-1EP_4x4mm_P0.5mm_EP2.5x2.5mm_ThermalVias
- removed the U2 at (18.6, 78.0)
- removed the U4 at (24.1, 78.0)
- removed U6: USBLC6-4SC6, Package_TO_SOT_SMD:SOT-23-6
- removed U7: MIC5528, Package_DFN_QFN:TDFN-6-1EP_2.5x2.5mm_P0.65mm_EP1.3x2mm_ThermalVias
- removed Y1: 25MHZ 18uF, Crystal:Crystal_SMD_5032-4Pin_5.0x3.2mm
Other:
- board outline added: 89 x 60.8 mm

Commit message: KiCad: update NavKF
Parts:
- moved U3 13.2 mm to (57.2, 121.5)
Changed lines of the file:
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@@
 	(footprint "Package_QFP:LQFP-144_20x20mm_P0.5mm"
 		(layer "F.Cu")
-		(at 62.25 133.6625)
+		(at 57.25 121.5)
 		(descr "LQFP, 144 Pin (JEDEC MS-026 variation BFB, 1.40mm body thickness, https://www.jedec.org/document_search?search_api_views_fulltext=MS-026, https://ww1.microchip.com/downloads/en/PackagingSpec/00000049BQ.pdf#page=425)")
 		(tags "LQFP QFP Microchip_144-Lead-Plastic-Low-Profile-Quad-Flatpack-(PL) Microsemi_TQ144")

Commit message: KiCad: update NavKF
[Version: v1.0.2] [Date: 2026-05-07T15:10:53+03:00]
Parts:
- moved U3 8.02 mm to (62.8, 115.7)
Changed lines of the file:
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@@
 	(footprint "Package_QFP:LQFP-144_20x20mm_P0.5mm"
 		(layer "F.Cu")
-		(at 57.25 121.5)
+		(at 62.75 115.6625)
 		(descr "LQFP, 144 Pin (JEDEC MS-026 variation BFB, 1.40mm body thickness, https://www.jedec.org/document_search?search_api_views_fulltext=MS-026, https://ww1.microchip.com/downloads/en/PackagingSpec/00000049BQ.pdf#page=425)")
 		(tags "LQFP QFP Microchip_144-Lead-Plastic-Low-Profile-Quad-Flatpack-(PL) Microsemi_TQ144")

Commit message: Chore: project cleanup
[Revision: REV-15] [Date: 2026-05-08 17:35:14]
Parts:
- moved U3 10.8 mm to (57.8, 125.2)
Changed lines of the file:
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@@
 	(footprint "Package_QFP:LQFP-144_20x20mm_P0.5mm"
 		(layer "F.Cu")
-		(at 62.75 115.6625)
+		(at 57.75 125.25)
 		(descr "LQFP, 144 Pin (JEDEC MS-026 variation BFB, 1.40mm body thickness, https://www.jedec.org/document_search?search_api_views_fulltext=MS-026, https://ww1.microchip.com/downloads/en/PackagingSpec/00000049BQ.pdf#page=425)")
 		(tags "LQFP QFP Microchip_144-Lead-Plastic-Low-Profile-Quad-Flatpack-(PL) Microsemi_TQ144")
